File: pcb2/shpad.kicad_pcb (KiCad board)
At the start: 2 copper layers, 60 x 53 mm, 12 parts, among them SW1 SW_Push, SW2 SW_Push, SW3 SW_Push, SW4 SW_Push, SW5 SW_Push, SW6 SW_Push, U1 MOUDLE-SEEEDUINO-XIAO, U2 ER_OLEDM0.91_1x-I2C

Commit message: Added images, added improved V2 of shpad edited readme
Parts:
- added G***: LOGO, LOGO, F.Cu at (59.5, 98.8)
- added G***: LOGO, LOGO, B.Cu at (38.0, 76.8)
- moved SW6 5.86 mm to (78.5, 108.8), turned to 180 degrees
- moved SW1 5.76 mm to (78.5, 89.8), turned to 0 degrees
- moved SW3 5.75 mm to (40.0, 89.8), turned to 0 degrees
- moved SW5 5.66 mm to (59.2, 108.8), turned to 180 degrees
- moved SW2 5.51 mm to (59.2, 89.5), turned to 0 degrees
- moved SW4 5.45 mm to (40.2, 108.8), turned to 180 degrees
Routing:
- net Net-(U1-PA02_A0_D0): track 54.5 -> 0.04 mm, vias 2 -> 0
- net GND: track 173.1 -> 220.7 mm
- net Net-(U1-PB09_A7_D7_RX): track 40.4 -> 59.7 mm, vias 2 -> 0
- net Net-(U1-PA7_A8_D8_SCK): track 39.9 -> 24.9 mm
- net Net-(U1-PA6_A10_D10_MOSI): track 17.2 -> 25.8 mm, vias 0 -> 1
- net Net-(U1-PA5_A9_D9_MISO): track 21.8 -> 13.9 mm, vias 3 -> 0
- net Net-(U1-PA4_A1_D1): track 61.0 -> 57.9 mm, vias 0 -> 1
Other:
- board size 60 x 53 mm -> 60 x 58.5 mm
- board text added: "Designed,coded and loved by naver"
